Commit message: fix: scale of urdf

File: golfcart_description/urdf/vehicle.xacro (robot description, xacro)
@@ -8,5 +8,5 @@
       <origin xyz="0 0 0" rpy="0 0 0"/>
       <geometry>
-        <mesh filename="package://golfcart_description/mesh/golfcart.dae" scale="1 1 1"/>
+        <mesh filename="package://golfcart_description/mesh/golfcart.dae" scale="1.4325 1.2091 1.1978"/>
       </geometry>
     </visual>
